File: BsidesRock2019.sch (KiCad schematic (older format))
At the start: 26 parts, among them U1 ATtiny85V-10SU

Commit message: Add files via upload
updated routes to pwn pins and ordered designs
Parts:
- removed C100uF1: CP1_Small, Capacitor_SMD:CP_Elec_6.3x5.4_Nichicon, symbol Device:CP1_Small
- removed SW-LEDGROUND1: SW_SPST, Button_Switch_SMD:SW_SPST_EVQPE1, symbol Switch:SW_SPST
Changed lines of the file:
@@
-$EndComp
-$Comp
-L Switch:SW_SPST SW-LEDGROUND1
-U 1 1 5BEA66B7
-P 3900 3650
-F 0 "SW-LEDGROUND1" H 3900 3885 50  0000 C CNN
-F 1 "SW_SPST" H 3900 3794 50  0000 C CNN
-F 2 "Button_Switch_SMD:SW_SPST_EVQPE1" H 3900 3650 50  0001 C CNN
-F 3 "" H 3900 3650 50  0001 C CNN
-	1    3900 3650
-	1    0    0    -1
 $EndComp
 $Comp
@@
 Connection ~ 2700 3800
 Wire Wire Line
-	3700 3650 3450 3650
-$Comp
-L Device:CP1_Small C100uF1
-U 1 1 5BEA6EFF
-P 2300 3150
-F 0 "C100uF1" H 2391 3196 50  0000 L CNN
-F 1 "CP1_Small" H 2391 3105 50  0000 L CNN
-F 2 "Capacitor_SMD:CP_Elec_6.3x5.4_Nichicon" H 2300 3150 50  0001 C CNN
-F 3 "~" H 2300 3150 50  0001 C CNN
-	1    2300 3150
-	1    0    0    -1
-$EndComp
-Wire Wire Line
 	1950 3500 1950 3300
 Wire Wire Line
 	1950 3300 2300 3300
-Wire Wire Line
-	2300 3300 2300 3250
 Wire Wire Line
 	2700 3500 2700 3300
@@
 Wire Wire Line
 	3350 3800 4100 3800
+Wire Wire Line
+	3450 3650 4100 3650
+Wire Wire Line
+	2300 3050 2300 3300
 $EndSCHEMATC
